File: schematic/kicad/ligma_ESP32-C3_economy_PEX_redesign_TI_charging.kicad_sch (KiCad schematic)
At the start: 107 parts, among them J1 ipex4, Q1 Q_PMOS_GSD, Q2 Q_NPN_BEC, Q3 Q_NPN_BEC, Q4 Q_PMOS_GSD, Q5 Q_PMOS_GSD, SW1 EVQ-P7A01P, SW2 EVQ-P7A01P, U1 USB_B_Micro, U2 TX4310-3V3, U3 LTC4054ES5-4.2, U4 BQ51013BRHLR, U5 ESP32-C3FH4, Y1 40MHz, Y2 32.768kHz

Commit message: add project images
Connections:
- net +BATT: now also SW1.2, SW1.2*
- net MainPower: no longer SW1.2, SW1.2*
Changed lines of the file:
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@@
   (junction (at 153.67 124.46) (diameter 0) (color 0 0 0 0)
   )
+  (junction (at 59.69 264.16) (diameter 0) (color 0 0 0 0)
+  )
   (junction (at 342.9 123.19) (diameter 0) (color 0 0 0 0)
   )
@@
   (junction (at 157.48 231.14) (diameter 0) (color 0 0 0 0)
   )
-  (junction (at 171.45 273.05) (diameter 0) (color 0 0 0 0)
-  )
   (junction (at 97.79 147.32) (diameter 0) (color 0 0 0 0)
   )
@@
   (junction (at 382.27 85.09) (diameter 0) (color 0 0 0 0)
   )
+  (junction (at 130.81 275.59) (diameter 0) (color 0 0 0 0)
+  )
   (junction (at 182.88 377.19) (diameter 0) (color 0 0 0 0)
-  )
-  (junction (at 130.81 273.05) (diameter 0) (color 0 0 0 0)
   )
   (junction (at 85.09 231.14) (diameter 0) (color 0 0 0 0)
@@
     (stroke (width 0) (type default) (color 0 0 0 0))
   )
-  (wire (pts (xy 59.69 262.89) (xy 59.69 273.05))
+  (wire (pts (xy 59.69 262.89) (xy 59.69 264.16))
     (stroke (width 0) (type default) (color 0 0 0 0))
   )
@@
     (stroke (width 0) (type default) (color 0 0 0 0))
   )
-  (wire (pts (xy 171.45 273.05) (xy 171.45 290.83))
-    (stroke (width 0) (type default) (color 0 0 0 0))
-  )
   (wire (pts (xy 77.47 119.38) (xy 99.06 119.38))
     (stroke (width 0) (type default) (color 0 0 0 0))
@@
     (stroke (width 0) (type default) (color 0 0 0 0))
   )
-  (wire (pts (xy 130.81 273.05) (xy 171.45 273.05))
-    (stroke (width 0) (type default) (color 0 0 0 0))
-  )
   (wire (pts (xy 205.74 220.98) (xy 205.74 231.14))
     (stroke (width 0) (type default) (color 0 0 0 0))
@@
     (stroke (width 0) (type default) (color 0 0 0 0))
   )
-  (wire (pts (xy 130.81 273.05) (xy 130.81 290.83))
-    (stroke (width 0) (type default) (color 0 0 0 0))
-  )
   (wire (pts (xy 473.71 135.89) (xy 473.71 137.16))
     (stroke (width 0) (type default) (color 0 0 0 0))
@@
     (stroke (width 0) (type default) (color 0 0 0 0))
   )
+  (wire (pts (xy 130.81 275.59) (xy 130.81 264.16))
+    (stroke (width 0) (type default) (color 0 0 0 0))
+  )
   (wire (pts (xy 128.27 353.06) (xy 128.27 354.33))
     (stroke (width 0) (type default) (color 0 0 0 0))
@@
     (stroke (width 0) (type default) (color 0 0 0 0))
   )
+  (wire (pts (xy 171.45 275.59) (xy 130.81 275.59))
+    (stroke (width 0) (type default) (color 0 0 0 0))
+  )
   (wire (pts (xy 121.92 177.8) (xy 130.81 177.8))
     (stroke (width 0) (type default) (color 0 0 0 0))
@@
     (stroke (width 0) (type default) (color 0 0 0 0))
   )
+  (wire (pts (xy 130.81 264.16) (xy 59.69 264.16))
+    (stroke (width 0) (type default) (color 0 0 0 0))
+  )
   (wire (pts (xy 157.48 220.98) (xy 157.48 231.14))
     (stroke (width 0) (type default) (color 0 0 0 0))
@@
     (stroke (width 0) (type default) (color 0 0 0 0))
   )
+  (wire (pts (xy 59.69 264.16) (xy 59.69 273.05))
+    (stroke (width 0) (type default) (color 0 0 0 0))
+  )
   (wire (pts (xy 92.71 213.36) (xy 101.6 213.36))
     (stroke (width 0) (type default) (color 0 0 0 0))
@@
     (stroke (width 0) (type default) (color 0 0 0 0))
   )
-  (wire (pts (xy 95.25 273.05) (xy 130.81 273.05))
-    (stroke (width 0) (type default) (color 0 0 0 0))
-  )
   (wire (pts (xy 116.84 177.8) (xy 116.84 124.46))
     (stroke (width 0) (type default) (color 0 0 0 0))
@@
     (stroke (width 0) (type default) (color 0 0 0 0))
   )
+  (wire (pts (xy 130.81 275.59) (xy 130.81 290.83))
+    (stroke (width 0) (type default) (color 0 0 0 0))
+  )
   (wire (pts (xy 354.33 123.19) (xy 342.9 123.19))
     (stroke (width 0) (type default) (color 0 0 0 0))
@@
     (stroke (width 0) (type default) (color 0 0 0 0))
   )
+  (wire (pts (xy 171.45 290.83) (xy 171.45 275.59))
+    (stroke (width 0) (type default) (color 0 0 0 0))
+  )
   (wire (pts (xy 33.02 135.89) (xy 39.37 135.89))
     (stroke (width 0) (type default) (color 0 0 0 0))
@@
     (stroke (width 0) (type default) (color 0 0 0 0))
   )
-  (wire (pts (xy 171.45 273.05) (xy 199.39 273.05))
+  (wire (pts (xy 95.25 273.05) (xy 199.39 273.05))
     (stroke (width 0) (type default) (color 0 0 0 0))
   )
@@
     (effects (font (size 1.27 1.27)) (justify left bottom))
   )
-  (text "long press soft toggle w/ momentary GPIO" (at 81.28 266.7 0)
+  (text "long press soft toggle w/ momentary GPIO" (at 82.55 261.62 0)
     (effects (font (size 2.54 2.54)) (justify left bottom))
   )
